File: AuxIO.kicad_sch (KiCad schematic)
At the start: 0 parts

Commit message: Latest updates
Parts:
- added J10: Conn_02x15_Odd_Even, symbol Connector_Generic:Conn_02x15_Odd_Even
Connections:
- new net GND: J10.7 (Pin_7), J10.8 (Pin_8)
- new net PA10(TIM1_CH3): J10.5 (Pin_5)
- new net PA8(TIM1_CH1): J10.1 (Pin_1)
- new net PA9(TIM1_CH2): J10.3 (Pin_3)
- new net PB13(TIM1_CH1N): J10.2 (Pin_2)
- new net PB14(TIM1_CH2N): J10.4 (Pin_4)
- new net PB15(TIM1_CH3N): J10.6 (Pin_6)
