File: PowerConverter.kicad_sch (KiCad schematic)
At the start: 0 parts

Commit message: Add files via upload
Parts:
- added C1: 180uF 35V, symbol Device:C_US
- added C2: 105, symbol Device:C
- added C3: 470uF 35V, symbol Device:C_US
- added C4, C5: 10µF, symbol Device:C_US
- added D1: 1N5821, Diode_THT:D_DO-201AD_P15.24mm_Horizontal, symbol Diode:1N5821
- added L1: L1 68uH/2A, symbol Device:L
- added R1: 100K, symbol Device:R_Small_US
- added U1: XL1509-5.0, Package_SO:SOIC-8_3.9x4.9mm_P1.27mm, symbol Regulator_Switching:XL1509-5.0
- added U2: AMS1117-3.3, Package_TO_SOT_SMD:SOT-223-3_TabPin2, symbol Regulator_Linear:AMS1117-3.3
Connections:
- new net: C2.1, C3.1, R1.1, U1.1 (VIN)
- new net: C1.2, C2.2, C3.2, C4.2, C5.2, D1.2 (A), U2.1 (GND)
- new net: D1.1 (K), L1.1, U1.2 (OUT)
- new net: R1.2, U1.4 (~{EN})
- new net +3V3 REG: C5.1, U2.2 (VO)
- new net FB: C1.1, C4.1, L1.2, U1.3 (FB), U2.3 (VI)
- new net GND: U1.5 (GND), U1.6 (GND), U1.7 (GND), U1.8 (GND)

Commit message: Latest updates
Parts:
- removed C1: 180uF 35V, symbol Device:C_US
- removed C2: 105, symbol Device:C
- removed C3: 470uF 35V, symbol Device:C_US
- removed C4, C5: 10µF, symbol Device:C_US
- removed D1: 1N5821, Diode_THT:D_DO-201AD_P15.24mm_Horizontal, symbol Diode:1N5821
- removed L1: L1 68uH/2A, symbol Device:L
- removed R1: 100K, symbol Device:R_Small_US
- removed U1: XL1509-5.0, Package_SO:SOIC-8_3.9x4.9mm_P1.27mm, symbol Regulator_Switching:XL1509-5.0
- removed U2: AMS1117-3.3, Package_TO_SOT_SMD:SOT-223-3_TabPin2, symbol Regulator_Linear:AMS1117-3.3
- added C18: 100uF-35V, Capacitor_THT:CP_Radial_D6.3mm_P2.50mm, symbol Device:C_Polarized
- added C19: 1u-50V, Capacitor_SMD:C_1206_3216Metric_Pad1.33x1.80mm_HandSolder, symbol Device:C
- added C20: 180uF-10V, Capacitor_THT:CP_Radial_D6.3mm_P2.50mm, symbol Device:C_Polarized
- added C21, C22: 10u, Capacitor_SMD:C_1206_3216Metric_Pad1.33x1.80mm_HandSolder, symbol Device:C
- added D4: SS34_C8678, EasyEDA:SMA_L4.3-W2.6-LS5.2-RD, symbol EasyEDA:SS34_C8678
- added L1: SMMS0650-680M, EasyEDA:IND-SMD_L7.1-W6.6_H5.0, symbol EasyEDA:SMMS0650-680M
- added U4: XL1509-5.0E1, EasyEDA:SOIC-8_L5.0-W4.0-P1.27-LS6.0-BL, symbol EasyEDA:XL1509-5.0E1
- added U5: AMS1117-3.3, LibMain:SOT-223-3_TabPin2_NOSILKSCREEN, symbol Regulator_Linear:AMS1117-3.3
Connections:
- net GND: now also C18.2, C19.2, C20.2, C21.2, C22.2, D4.2 (A), U4.5 (GND), U4.6 (GND), U4.7 (GND), U4.8 (GND), U5.1 (GND)
- new net: D4.1 (K), L1.1, U4.2 (OUTPUT)
- new net +12V: C18.1, C19.1, U4.1 (VIN)
- new net +3.3V: C22.1, U5.2 (VO)
- new net +5V: C20.1, C21.1, L1.2, U4.3 (FB), U5.3 (VI)
- no-connect marks 0 -> 1
Other:
- note added: "BUCK"
- note added: "LDO"

Commit message: Schematic--Footprint link
Parts:
- U5: footprint LibMain:SOT-223-3_TabPin2_NOSILKSCREEN -> Package_TO_SOT_SMD:SOT-223-3_TabPin2
Changed lines of the file:
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@@
 			)
 		)
-		(property "Footprint" "LibMain:SOT-223-3_TabPin2_NOSILKSCREEN"
+		(property "Footprint" "Package_TO_SOT_SMD:SOT-223-3_TabPin2"
 			(at 227.33 72.39 0)
 			(effects
